File: flypanels/flypanels.sch (KiCad schematic (older format))
At the start: 17 parts, among them IC1 ATMEGA168-A, P1 CONN_8, P2 CONN_8, U1 ULN2804A, X1 CER_RESO

Commit message: file cleanup
Parts:
- C1, C2: symbol C -> flypanels-rescue:C
- IC1: symbol ATMEGA168-A -> flypanels-rescue:ATMEGA168-A
- MATRIX1: symbol LED_8X8 -> flypanels-rescue:LED_8X8
- P1, P2: symbol CONN_8 -> flypanels-rescue:CONN_8
- R1, R2, R3, R4, R5, R6, R7, R8, R9: symbol R -> flypanels-rescue:R
- U1: symbol ULN2804A -> flypanels-rescue:ULN2804A
- X1: symbol CER_RESO -> flypanels-rescue:CER_RESO
